File: choc_v1/pearbear_choc.kicad_pcb (KiCad board)
At the start: 2 copper layers, 117.5 x 68 mm, 26 parts, among them J1 rj11, SW1 SW_Push, SW10 SW_Push, SW11 SW_Push, SW12 SW_Push, SW13 SW_Push, SW14 SW_Push, SW15 SW_Push, SW16 SW_Push, SW17 SW_Push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

Commit message: choc
Parts:
- moved SW1 2.94 mm to (103.8, 88.2)
- moved SW11 2.94 mm to (109.3, 122.2)
- moved SW6 2.94 mm to (106.6, 105.2)
- moved SW_Reset1 0.55 mm to (103.8, 70.2)
Routing:
- net Switch11: track 108.0 -> 109.8 mm
- net Switch6: track 100.8 -> 102.0 mm
- net Switch1: track 100.8 -> 102.0 mm
- net reset: track 126.9 -> 127.5 mm
Changed lines of the file:
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@@
 	(title_block
 		(title "pearbear_choc")
-		(date "2024-10-08")
+		(date "2025-02-09")
 		(rev "1")
 		(company "tomsadowski")
@@
 	(footprint "pb_fb:SW_Kailh_Choc_v1_reversible"
 		(layer "F.Cu")
-		(at 103.79 85.275)
+		(at 103.79 88.215)
 		(descr "Compatible with Cherry MX Low Profile, Kailh Choc V1 (PG1350) and Choc V2 (PG1353) low profile mechanical keyboard switch, through-hole soldering, single-sided mounting.")
 		(tags "switch, low_profile")
@@
 	(footprint "pb_fb:SW_Kailh_Choc_v1_reversible"
 		(layer "F.Cu")
-		(at 109.33 119.275)
+		(at 109.33 122.215)
 		(descr "Compatible with Cherry MX Low Profile, Kailh Choc V1 (PG1350) and Choc V2 (PG1353) low profile mechanical keyboard switch, through-hole soldering, single-sided mounting.")
 		(tags "switch, low_profile")
@@
 	(footprint "pb_fb:SW_TH_Tactile_Omron_B3F-10xx_reversible"
 		(layer "F.Cu")
-		(at 103.79 70.747)
+		(at 103.79 70.2)
 		(descr "SW_TH_Tactile_Omron_B3F-10xx_https://www.omron.com/ecb/products/pdf/en-b3f.pdf")
 		(tags "Omron B3F-10xx")
@@
 	(footprint "pb_fb:SW_Kailh_Choc_v1_reversible"
 		(layer "F.Cu")
-		(at 106.56 102.275)
+		(at 106.56 105.215)
 		(descr "Compatible with Cherry MX Low Profile, Kailh Choc V1 (PG1350) and Choc V2 (PG1353) low profile mechanical keyboard switch, through-hole soldering, single-sided mounting.")
 		(tags "switch, low_profile")
@@
 	)
 	(gr_text "pearbear_choc"
-		(at 97.56 119.275 90)
+		(at 97.83 122.215 90)
 		(layer "B.SilkS")
 		(effects
@@
 	)
 	(gr_text "pearbear_choc"
-		(at 97.56 119.275 90)
+		(at 97.83 122.215 90)
 		(layer "F.SilkS")
 		(effects
@@
 	)
 	(segment
-		(start 107.04 72.997)
-		(end 107.052 72.997)
+		(start 119.37 95.78)
+		(end 186.93802 95.78)
 		(width 0.25)
 		(layer "B.Cu")
@@
 	)
 	(segment
-		(start 114.25 90.66)
-		(end 119.37 95.78)
-		(width 0.25)
-		(layer "B.Cu")
-		(net 1)
-	)
-	(segment
-		(start 190.79 91.92802)
-		(end 190.79 82.66)
+		(start 107.04 72.45)
+		(end 114.25 79.66)
 		(width 0.25)
 		(layer "B.Cu")
@@
 	)
 	(segment
-		(start 114.25 80.195)
-		(end 114.25 90.66)
+		(start 107.04 72.45)
+		(end 100.54 72.45)
 		(width 0.25)
 		(layer "B.Cu")
@@
 	)
 	(segment
-		(start 119.37 95.78)
-		(end 186.93802 95.78)
+		(start 186.93802 95.78)
+		(end 190.79 91.92802)
 		(width 0.25)
 		(layer "B.Cu")
@@
 	)
 	(segment
-		(start 107.04 72.997)
-		(end 100.54 72.997)
+		(start 114.25 90.66)
+		(end 119.37 95.78)
 		(width 0.25)
 		(layer "B.Cu")
@@
 	)
 	(segment
-		(start 186.93802 95.78)
-		(end 190.79 91.92802)
+		(start 114.25 79.66)
+		(end 114.25 90.66)
 		(width 0.25)
 		(layer "B.Cu")
@@
 	)
 	(segment
-		(start 107.052 72.997)
-		(end 114.25 80.195)
+		(start 190.79 91.92802)
+		(end 190.79 82.66)
 		(width 0.25)
 		(layer "B.Cu")
@@
 	)
 	(segment
-		(start 191.24 92.114416)
-		(end 187.124416 96.23)
+		(start 187.124416 96.23)
+		(end 109.645 96.23)
 		(width 0.25)
 		(layer "B.Cu")
@@
 	)
 	(segment
-		(start 196.684 81.37)
-		(end 195.394 82.66)
+		(start 109.645 96.23)
+		(end 106.56 99.315)
 		(width 0.25)
 		(layer "B.Cu")
@@
 	)
 	(segment
-		(start 195.394 82.66)
-		(end 193.145 82.66)
+		(start 191.24 92.114416)
+		(end 187.124416 96.23)
 		(width 0.25)
 		(layer "B.Cu")
@@
 	)
 	(segment
-		(start 191.24 84.565)
-		(end 191.24 92.114416)
+		(start 195.394 82.66)
+		(end 193.145 82.66)
 		(width 0.25)
 		(layer "B.Cu")
@@
 	)
 	(segment
-		(start 106.705 96.23)
-		(end 106.56 96.375)
+		(start 191.24 84.565)
+		(end 191.24 92.114416)
 		(width 0.25)
 		(layer "B.Cu")
@@
 	)
 	(segment
-		(start 187.124416 96.23)
-		(end 106.705 96.23)
+		(start 196.684 81.37)
+		(end 195.394 82.66)
 		(width 0.25)
 		(layer "B.Cu")
@@
 	)
 	(segment
-		(start 111.37 113.375)
-		(end 109.33 113.375)
+		(start 116.38 108.365)
+		(end 109.33 115.415)
 		(width 0.25)
 		(layer "B.Cu")
@@
 	)
 	(segment
-		(start 187.310812 96.68)
-		(end 119.495 96.68)
+		(start 195.354 85.24)
+		(end 192.85 85.24)
 		(width 0.25)
 		(layer "B.Cu")
@@
 	)
 	(segment
-		(start 119.495 96.68)
-		(end 116.38 99.795)
+		(start 192.85 85.24)
+		(end 191.69 86.4)
 		(width 0.25)
 		(layer "B.Cu")
@@
 	)
 	(segment
-		(start 191.69 92.300812)
-		(end 187.310812 96.68)
+		(start 116.38 99.795)
+		(end 116.38 108.365)
 		(width 0.25)
 		(layer "B.Cu")
@@
 	)
 	(segment
-		(start 192.85 85.24)
-		(end 191.69 86.4)
+		(start 187.310812 96.68)
+		(end 119.495 96.68)
 		(width 0.25)
 		(layer "B.Cu")
@@
 	)
 	(segment
-		(start 116.38 99.795)
-		(end 116.38 108.365)
+		(start 191.69 86.4)
+		(end 191.69 92.300812)
 		(width 0.25)
 		(layer "B.Cu")
@@
 	)
 	(segment
-		(start 116.38 108.365)
-		(end 111.37 113.375)
+		(start 191.69 92.300812)
+		(end 187.310812 96.68)
 		(width 0.25)
 		(layer "B.Cu")
@@
 	)
 	(segment
-		(start 191.69 86.4)
-		(end 191.69 92.300812)
+		(start 119.495 96.68)
+		(end 116.38 99.795)
 		(width 0.25)
 		(layer "B.Cu")
@@
 	)
 	(segment
-		(start 195.354 85.24)
-		(end 192.85 85.24)
+		(start 109.33 115.415)
+		(end 109.33 116.315)
 		(width 0.25)
 		(layer "B.Cu")
@@
 	)
 	(segment
-		(start 104.57 78.595)
-		(end 125.743604 78.595)
+		(start 195.414 90.26)
+		(end 196.684 88.99)
 		(width 0.25)
 		(layer "F.Cu")
@@
 	)
 	(segment
-		(start 193.27 90.26)
-		(end 195.414 90.26)
+		(start 182.112792 79.375)
+		(end 183.837792 81.1)
 		(width 0.25)
 		(layer "F.Cu")
@@
 	)
 	(segment
-		(start 103.79 79.375)
-		(end 104.57 78.595)
+		(start 125.743604 78.595)
+		(end 126.523604 79.375)
 		(width 0.25)
 		(layer "F.Cu")
@@
 	)
 	(segment
-		(start 183.837792 81.1)
-		(end 187.917208 81.1)
+		(start 192.02 85.202792)
+		(end 192.02 89.01)
 		(width 0.25)
 		(layer "F.Cu")
@@
 	)
 	(segment
-		(start 195.414 90.26)
-		(end 196.684 88.99)
+		(start 103.79 82.315)
+		(end 107.51 78.595)
 		(width 0.25)
 		(layer "F.Cu")
@@
 	)
 	(segment
-		(start 192.02 85.202792)
-		(end 192.02 89.01)
+		(start 192.02 89.01)
+		(end 193.27 90.26)
 		(width 0.25)
 		(layer "F.Cu")
@@
 	)
 	(segment
-		(start 182.112792 79.375)
-		(end 183.837792 81.1)
+		(start 187.917208 81.1)
+		(end 192.02 85.202792)
 		(width 0.25)
 		(layer "F.Cu")
@@
 	)
 	(segment
-		(start 126.523604 79.375)
-		(end 182.112792 79.375)
+		(start 193.27 90.26)
+		(end 195.414 90.26)
 		(width 0.25)
 		(layer "F.Cu")
@@
 	)
 	(segment
-		(start 192.02 89.01)
-		(end 193.27 90.26)
+		(start 126.523604 79.375)
+		(end 182.112792 79.375)
 		(width 0.25)
 		(layer "F.Cu")
@@
 	)
 	(segment
-		(start 125.743604 78.595)
-		(end 126.523604 79.375)
+		(start 183.837792 81.1)
+		(end 187.917208 81.1)
 		(width 0.25)
 		(layer "F.Cu")
@@
 	)
 	(segment
-		(start 187.917208 81.1)
-		(end 192.02 85.202792)
+		(start 107.51 78.595)
+		(end 125.743604 78.595)
 		(width 0.25)
 		(layer "F.Cu")
